File: hardware/fan-output.kicad_sch (KiCad schematic)
At the start: 7 parts, among them J5 Conn_01x04

Commit message: Start placement and routing
Parts:
- J9: renamed from J5; footprint (none) -> Homebrew:CONN-TH_47053-1000
- R29: renamed from R14; footprint Resistor_SMD:R_0603_1608Metric -> Resistor_SMD:R_0603_1608Metric_Pad0.98x0.95mm_HandSolder
- renumbered D5 to D19, D6 to D20, D4 to D21, R15 to R27, R13 to R28
Changed lines of the file:
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@@
 		(dnp no)
 		(fields_autoplaced yes)
-		(property "Reference" "D6"
+		(property "Reference" "D20"
 			(at 54.102 24.1878 90)
 			(effects
@@
 		(on_board yes)
 		(dnp no)
-		(property "Reference" "J5"
+		(property "Reference" "J9"
 			(at 76.962 38.0422 0)
 			(effects
@@
 			)
 		)
-		(property "Footprint" ""
+		(property "Footprint" "Homebrew:CONN-TH_47053-1000"
 			(at 74.93 38.1 0)
 			(effects
@@
 		(dnp no)
 		(fields_autoplaced yes)
-		(property "Reference" "R15"
+		(property "Reference" "R27"
 			(at 36.068 30.5378 0)
 			(effects
@@
 		(dnp no)
 		(fields_autoplaced yes)
-		(property "Reference" "R13"
+		(property "Reference" "R28"
 			(at 44.45 30.3995 90)
 			(effects
@@
 		(dnp no)
 		(fields_autoplaced yes)
-		(property "Reference" "R14"
+		(property "Reference" "R29"
 			(at 57.15 15.1595 90)
 			(effects
@@
 			)
 		)
-		(property "Footprint" "Resistor_SMD:R_0603_1608Metric"
+		(property "Footprint" "Resistor_SMD:R_0603_1608Metric_Pad0.98x0.95mm_HandSolder"
 			(at 57.15 22.098 90)
 			(effects
@@
 		(dnp no)
 		(fields_autoplaced yes)
-		(property "Reference" "D4"
+		(property "Reference" "D21"
 			(at 56.642 45.7778 90)
 			(effects
@@
 		(dnp no)
 		(fields_autoplaced yes)
-		(property "Reference" "#PWR032"
+		(property "Reference" "#PWR052"
 			(at 54.61 46.99 0)
 			(effects
@@
 		(dnp no)
 		(fields_autoplaced yes)
-		(property "Reference" "#PWR029"
+		(property "Reference" "#PWR046"
 			(at 39.37 49.53 0)
 			(effects
@@
 		(dnp no)
 		(fields_autoplaced yes)
-		(property "Reference" "#PWR028"
+		(property "Reference" "#PWR047"
 			(at 52.07 35.56 0)
 			(effects
@@
 		(dnp no)
 		(fields_autoplaced yes)
-		(property "Reference" "D5"
+		(property "Reference" "D19"
 			(at 41.402 38.1578 90)
 			(effects
@@
 		(dnp no)
 		(fields_autoplaced yes)
-		(property "Reference" "#PWR026"
+		(property "Reference" "#PWR049"
 			(at 34.29 31.75 0)
 			(effects

Commit message: Hardware v1.1
Parts:
- added C29: 10uF, Capacitor_SMD:C_0603_1608Metric, symbol Device:C
Connections:
- net +12V: now also C29.1
- net FAN_GND: now also C29.2
Other:
- moved on the sheet: D19, R27, R28
Changed lines of the file:
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@@
+	)
+	(junction
+		(at 54.61 50.8)
+		(diameter 0)
+		(color 0 0 0 0)
 	)
 	(junction
@@
 	)
 	(junction
-		(at 34.29 35.56)
+		(at 24.13 35.56)
 		(diameter 0)
 		(color 0 0 0 0)
@@
 	)
 	(junction
-		(at 39.37 35.56)
+		(at 29.21 35.56)
 		(diameter 0)
 		(color 0 0 0 0)
@@
 	(wire
 		(pts
-			(xy 39.37 35.56) (xy 40.64 35.56)
+			(xy 29.21 35.56) (xy 30.48 35.56)
 		)
 		(stroke
@@
 	(wire
 		(pts
-			(xy 48.26 35.56) (xy 69.85 35.56)
-		)
-		(stroke
-			(width 0)
-			(type default)
-		)
-	)
-	(wire
-		(pts
-			(xy 31.75 35.56) (xy 34.29 35.56)
+			(xy 38.1 35.56) (xy 69.85 35.56)
+		)
+		(stroke
+			(width 0)
+			(type default)
+		)
+	)
+	(wire
+		(pts
+			(xy 43.18 43.18) (xy 54.61 43.18)
+		)
+		(stroke
+			(width 0)
+			(type default)
+		)
+	)
+	(wire
+		(pts
+			(xy 21.59 35.56) (xy 24.13 35.56)
 		)
 		(stroke
@@
 	(wire
 		(pts
+			(xy 43.18 50.8) (xy 54.61 50.8)
+		)
+		(stroke
+			(width 0)
+			(type default)
+		)
+	)
+	(wire
+		(pts
 			(xy 66.04 33.02) (xy 69.85 33.02)
 		)
@@
 	(wire
 		(pts
-			(xy 34.29 35.56) (xy 39.37 35.56)
+			(xy 24.13 35.56) (xy 29.21 35.56)
 		)
 		(stroke
@@
 	(hierarchical_label "TACH"
 		(shape input)
-		(at 31.75 35.56 180)
+		(at 21.59 35.56 180)
 		(fields_autoplaced yes)
 		(effects
@@
 	(symbol
 		(lib_id "Device:R")
-		(at 34.29 31.75 180)
+		(at 24.13 31.75 180)
 		(unit 1)
 		(exclude_from_sim no)
@@
 		(fields_autoplaced yes)
 		(property "Reference" "R27"
-			(at 36.068 30.5378 0)
+			(at 25.908 30.5378 0)
 			(effects
 				(font
@@
 		)
 		(property "Value" "100k"
-			(at 36.068 32.9621 0)
+			(at 25.908 32.9621 0)
 			(effects
 				(font
@@
 		)
 		(property "Footprint" "Resistor_SMD:R_0603_1608Metric_Pad0.98x0.95mm_HandSolder"
-			(at 36.068 31.75 90)
+			(at 25.908 31.75 90)
 			(effects
 				(font
@@
 		)
 		(property "Datasheet" "~"
-			(at 34.29 31.75 0)
+			(at 24.13 31.75 0)
 			(effects
 				(font
@@
 		)
 		(property "Description" "Resistor"
-			(at 34.29 31.75 0)
+			(at 24.13 31.75 0)
 			(effects
 				(font
@@
 		)
 		(property "LCSC" "C25803"
-			(at 34.29 31.75 0)
+			(at 24.13 31.75 0)
 			(effects
 				(font
@@
 	(symbol
 		(lib_id "Device:R")
-		(at 44.45 35.56 90)
+		(at 34.29 35.56 90)
 		(unit 1)
 		(exclude_from_sim no)
@@
 		(fields_autoplaced yes)
 		(property "Reference" "R28"
-			(at 44.45 30.3995 90)
+			(at 34.29 30.3995 90)
 			(effects
 				(font
@@
 		)
 		(property "Value" "1k"
-			(at 44.45 32.8238 90)
+			(at 34.29 32.8238 90)
 			(effects
 				(font
@@
 		)
 		(property "Footprint" "Resistor_SMD:R_0402_1005Metric"
-			(at 44.45 37.338 90)
+			(at 34.29 37.338 90)
 			(effects
 				(font
@@
 		)
 		(property "Datasheet" "~"
-			(at 44.45 35.56 0)
+			(at 34.29 35.56 0)
 			(effects
 				(font
@@
 		)
 		(property "Description" "Resistor"
-			(at 44.45 35.56 0)
+			(at 34.29 35.56 0)
 			(effects
 				(font
@@
 		)
 		(property "LCSC" "C11702"
-			(at 44.45 35.56 0)
+			(at 34.29 35.56 0)
 			(effects
 				(font
@@
 	)
 	(symbol
+		(lib_id "Device:C")
+		(at 43.18 46.99 0)
+		(unit 1)
+		(exclude_from_sim no)
+		(in_bom yes)
+		(on_board yes)
+		(dnp no)
+		(fields_autoplaced yes)
+		(property "Reference" "C29"
+			(at 46.101 45.7778 0)
+			(effects
+				(font
+					(size 1.27 1.27)
+				)
+				(justify left)
+			)
+		)
+		(property "Value" "10uF"
+			(at 46.101 48.2021 0)
+			(effects
+				(font
+					(size 1.27 1.27)
+				)
+				(justify left)
+			)
+		)
+		(property "Footprint" "Capacitor_SMD:C_0603_1608Metric"
+			(at 44.1452 50.8 0)
+			(effects
+				(font
+					(size 1.27 1.27)
+				)
+				(hide yes)
+			)
+		)
+		(property "Datasheet" "~"
+			(at 43.18 46.99 0)
+			(effects
+				(font
+					(size 1.27 1.27)
+				)
+				(hide yes)
+			)
+		)
+		(property "Description" "Unpolarized capacitor"
+			(at 43.18 46.99 0)
+			(effects
+				(font
+					(size 1.27 1.27)
+				)
+				(hide yes)
+			)
+		)
+		(property "LCSC" "C96446"
+			(at 43.18 46.99 0)
+			(effects
+				(font
+					(size 1.27 1.27)
+				)
+				(hide yes)
+			)
+		)
+		(pin "1"
+		)
+		(pin "2"
+		)
+		(instances
+			(project "air-filter-controller"
+				(path "/507e7113-3c01-4251-b852-8c77f2a74b1d/3f730f89-203a-4ecf-9d39-ee2f2b8bb3bf"
+					(reference "C29")
+					(unit 1)
+				)
+				(path "/507e7113-3c01-4251-b852-8c77f2a74b1d/5cba8fe0-777e-4016-8937-7c62083b14bf"
+					(reference "C28")
+					(unit 1)
+				)
+				(path "/507e7113-3c01-4251-b852-8c77f2a74b1d/6494b452-a92a-4691-a65c-0df806c10a83"
+					(reference "C27")
+					(unit 1)
+				)
+				(path "/507e7113-3c01-4251-b852-8c77f2a74b1d/65717a82-319c-4318-812f-149098c14f8b"
+					(reference "C31")
+					(unit 1)
+				)
+				(path "/507e7113-3c01-4251-b852-8c77f2a74b1d/8937d470-f6df-4629-ba39-a1967a97857d"
+					(reference "C33")
+					(unit 1)
+				)
+				(path "/507e7113-3c01-4251-b852-8c77f2a74b1d/8c955da3-adc8-438b-b7c7-56a208f33014"
+					(reference "C26")
+					(unit 1)
+				)
+				(path "/507e7113-3c01-4251-b852-8c77f2a74b1d/9328a37d-03a3-4c63-b6b5-171b971693f4"
+					(reference "C25")
+					(unit 1)
+				)
+				(path "/507e7113-3c01-4251-b852-8c77f2a74b1d/b954c781-f82c-45af-826a-fbe5f85e7049"
+					(reference "C24")
+					(unit 1)
+				)
+				(path "/507e7113-3c01-4251-b852-8c77f2a74b1d/da5fa1d1-cc9e-4c4e-992a-b83a41aa2c60"
+					(reference "C32")
+					(unit 1)
+				)
+				(path "/507e7113-3c01-4251-b852-8c77f2a74b1d/ea19b6ef-b9dc-466f-baea-e01e683266f3"
+					(reference "C30")
+					(unit 1)
+				)
+			)
+		)
+	)
+	(symbol
 		(lib_id "power:GND")
-		(at 39.37 43.18 0)
+		(at 29.21 43.18 0)
 		(unit 1)
 		(exclude_from_sim no)
@@
 		(fields_autoplaced yes)
 		(property "Reference" "#PWR046"
-			(at 39.37 49.53 0)
+			(at 29.21 49.53 0)
 			(effects
 				(font
@@
 		)
 		(property "Value" "GND"
-			(at 39.37 47.3131 0)
+			(at 29.21 47.3131 0)
 			(effects
 				(font
@@
 		)
 		(property "Footprint" ""
-			(at 39.37 43.18 0)
+			(at 29.21 43.18 0)
 			(effects
 				(font
@@
 		)
 		(property "Datasheet" ""
-			(at 39.37 43.18 0)
+			(at 29.21 43.18 0)
 			(effects
 				(font
@@
 		)
 		(property "Description" "Power symbol creates a global label with name \"GND\" , ground"
-			(at 39.37 43.18 0)
+			(at 29.21 43.18 0)
 			(effects
 				(font
@@
 	(symbol
 		(lib_id "Device:D")
-		(at 39.37 39.37 270)
+		(at 29.21 39.37 270)
 		(unit 1)
 		(exclude_from_sim no)
@@
 		(fields_autoplaced yes)
 		(property "Reference" "D19"
-			(at 41.402 38.1578 90)
+			(at 31.242 38.1578 90)
 			(effects
 				(font
@@
 		)
 		(property "Value" "SMAJ5.0A"
-			(at 41.402 40.5821 90)
+			(at 31.242 40.5821 90)
 			(effects
 				(font
@@
 		)
 		(property "Footprint" "Diode_SMD:D_SMA"
-			(at 39.37 39.37 0)
+			(at 29.21 39.37 0)
 			(effects
 				(font
@@
 		)
 		(property "Datasheet" "~"
-			(at 39.37 39.37 0)
+			(at 29.21 39.37 0)
 			(effects
 				(font
@@
 		)
 		(property "Description" "Diode"
-			(at 39.37 39.37 0)
+			(at 29.21 39.37 0)
 			(effects
 				(font
@@
 		)
 		(property "Sim.Device" "D"
-			(at 39.37 39.37 0)
+			(at 29.21 39.37 0)
 			(effects
 				(font
@@
 		)
 		(property "Sim.Pins" "1=K 2=A"
-			(at 39.37 39.37 0)
+			(at 29.21 39.37 0)
 			(effects
 				(font
@@
 		)
 		(property "MPN" "SMAJ5.0A"
-			(at 39.37 39.37 90)
+			(at 29.21 39.37 90)
 			(effects
 				(font
@@
 		)
 		(property "LCSC" "C113952"
-			(at 39.37 39.37 90)
+			(at 29.21 39.37 90)
 			(effects
 				(font
@@
 	(symbol
 		(lib_id "power:+3V3")
-		(at 34.29 27.94 0)
+		(at 24.13 27.94 0)
 		(unit 1)
 		(exclude_from_sim no)
@@
 		(fields_autoplaced yes)
 		(property "Reference" "#PWR0110"
-			(at 34.29 31.75 0)
+			(at 24.13 31.75 0)
 			(effects
 				(font
@@
 		)
 		(property "Value" "+3V3"
-			(at 34.29 23.8069 0)
+			(at 24.13 23.8069 0)
 			(effects
 				(font
@@
 		)
 		(property "Footprint" ""
-			(at 34.29 27.94 0)
+			(at 24.13 27.94 0)
 			(effects
 				(font
@@
 		)
 		(property "Datasheet" ""
-			(at 34.29 27.94 0)
+			(at 24.13 27.94 0)
 			(effects
 				(font
@@
 		)
 		(property "Description" "Power symbol creates a global label with name \"+3V3\""
-			(at 34.29 27.94 0)
-			(effects
-				(font
+			(at 24.13 27.94 0)
+			(effects
+				(font
